Commit message: feat: integrate dual-backend services and agent debugging workspace

File: assets/eyoubot/eu_ca_describtion_lbs6.urdf (robot description, URDF)
Before this commit: robot eu_ca_describtion_lbs6, 27 links, 26 joints
Links:
- link base_link: geometry collision mesh filename=meshes/SensorConnect.STL; visual mesh filename=meshes/SensorConnect.STL
